File: adda-blinky/adda-blinky.kicad_pcb (KiCad board)
At the start: 2 copper layers, 2 parts, among them U1 ATtiny1616-S, U2 ATtiny1616-M

Commit message: WIP add bus LEDs
Parts:
- added D0: LED, Diode_SMD:D_0805_2012Metric, F.Cu at (104.8, 74.5)
- added D1: LED, Diode_SMD:D_0805_2012Metric, F.Cu at (104.8, 71.5)
- added D2: LED, Diode_SMD:D_0805_2012Metric, F.Cu at (104.8, 68.4)
- added D3: LED, Diode_SMD:D_0805_2012Metric, F.Cu at (104.8, 65.4)
- added D4: LED, Diode_SMD:D_0805_2012Metric, F.Cu at (104.8, 62.3)
- added D5: LED, Diode_SMD:D_0805_2012Metric, F.Cu at (104.8, 59.3)
- added D6: LED, Diode_SMD:D_0805_2012Metric, F.Cu at (104.8, 56.3)
- added D7: LED, Diode_SMD:D_0805_2012Metric, F.Cu at (104.8, 53.2)
Connections:
- net Net-(U2-Pad1) renamed /PA2
- net Net-(U2-Pad10) renamed /PB4
- net Net-(U2-Pad11) renamed /PB3
- net Net-(U2-Pad12) renamed /PB2
- net Net-(U2-Pad13) renamed /PB1
- net Net-(U2-Pad14) renamed /PB0
- net Net-(U2-Pad15) renamed /PC0
- net Net-(U2-Pad16) renamed /PC1
- net Net-(U2-Pad17) renamed /PC2
- net Net-(U2-Pad18) renamed /PC3
- net Net-(U2-Pad19) renamed /PA0
- net Net-(U2-Pad2) renamed /PA3
- net Net-(U2-Pad20) renamed /PA1
- net Net-(U2-Pad21) renamed GND
- net Net-(U2-Pad4) renamed +3.3V
- net Net-(U2-Pad5) renamed /PA4
- net Net-(U2-Pad6) renamed /PA5
- net Net-(U2-Pad7) renamed /PA6
- net Net-(U2-Pad8) renamed /PA7
- net Net-(U2-Pad9) renamed /PB5
Routing:
- net GND: track 0.00 -> 8.10 mm
- net /PA3: track 0.00 -> 5.69 mm
- net /PA2: track 0.00 -> 4.59 mm

Commit message: WIP
Parts:
- added C1: 1u, Capacitor_SMD:C_0805_2012Metric, F.Cu at (114.5, 52.5)
- added C2: 1u, Capacitor_SMD:C_0805_2012Metric, F.Cu at (112.5, 52.5)
- added J1: Conn_01x02, Connector_Molex:Molex_KK-254_AE-6410-02A_1x02_P2.54mm_Vertical, F.Cu at (104.6, 59.3)
- added J2: Conn_01x02, Connector_Molex:Molex_KK-254_AE-6410-02A_1x02_P2.54mm_Vertical, F.Cu at (104.6, 66.9)
- added J3: USB_B_Micro, Connector_USB:USB_Micro-AB_Molex_47590-0001, F.Cu at (137.8, 61.2)
- added J4: Conn_01x02, Connector_Molex:Molex_KK-254_AE-6410-02A_1x02_P2.54mm_Vertical, F.Cu at (104.6, 51.7)
- added U3: AMS1117-3.3, Package_TO_SOT_SMD:SOT-223-3_TabPin2, F.Cu at (121.4, 51.7)
- moved D7 23.6 mm to (114.0, 75.0), turned to -90 degrees
- moved D0 23.5 mm to (128.3, 74.9), turned to -90 degrees
- moved D6 21.8 mm to (116.1, 75.0), turned to -90 degrees
- moved D1 21.7 mm to (126.2, 74.9), turned to -90 degrees
- moved D5 20.6 mm to (118.1, 75.0), turned to -90 degrees
- moved D2 20.5 mm to (124.2, 75.0), turned to -90 degrees
- moved D4 19.9 mm to (120.1, 75.0), turned to -90 degrees
- moved D3 19.8 mm to (122.2, 75.0), turned to -90 degrees
Connections:
- net /PA0 renamed /~{RESET}
- net /PA1 renamed /PA1/MOSI/SDA
- net /PA2 renamed /PA2/MISO/SCL
- net /PA3 renamed /PA3/SCK
- net /PA4 renamed /PA4/SS
- net /PA5 renamed /PA5/AIN5
- net /PA6 renamed /PA6/OUT
- D0 pad 1: /PB0 -> /PC0
- D1 pad 1: /PB1 -> /PC1
- D2 pad 1: /PB2 -> /PC2
- D3 pad 1: /PB3 -> /PC3
- D4 pad 1: /PB4 -> /PB0
- D5 pad 1: /PB5 -> /PB1
- D6 pad 1: unconnected-(D6-K-Pad1) -> /PB2
- D7 pad 1: unconnected-(D7-K-Pad1) -> /PB3
Routing:
- net /PC3: track 3.46 -> 17.5 mm, vias 0 -> 2
- net /PC2: track 3.82 -> 14.8 mm, vias 0 -> 2
- net /PC1: track 4.97 -> 13.3 mm, vias 0 -> 2
- net /PB3: track 4.85 -> 12.7 mm
- net /PB2: track 6.14 -> 13.3 mm
- net /PB0: track 6.85 -> 13.8 mm
- net /PC0: track 5.63 -> 12.5 mm
- net /PB1: track 7.58 -> 12.7 mm
- net GND: track 8.10 -> 10.9 mm, vias 0 -> 3
Other:
- board outline added: 46.2 x 35.1 mm
