File: adda-blinky/adda-blinky.kicad_sch (KiCad schematic)
At the start: 2 parts, among them U1 ATtiny1616-S, U2 ATtiny1616-M

Commit message: WIP add bus LEDs
Parts:
- added D0, D1, D2, D3, D4, D5, D6, D7: LED, Diode_SMD:D_0805_2012Metric, symbol Device:LED
Connections:
- net +3.3V: now reaches U1.1 (VCC), U2.4 (VCC)
- net +3.3V: now also D0.2 (A), D1.2 (A), D2.2 (A), D3.2 (A), D4.2 (A), D5.2 (A), D6.2 (A), D7.2 (A)
- net PB1: now reaches U1.10 (PB1), U2.13 (PB1)
- net PB1: now also D1.1 (K)
- net PB0: now reaches U1.11 (PB0), U2.14 (PB0)
- net PB0: now also D0.1 (K)
- net PC0: now reaches U1.12 (PC0), U2.15 (PC0)
- net PC1: now reaches U1.13 (PC1), U2.16 (PC1)
- net PC2: now reaches U1.14 (PC2), U2.17 (PC2)
- net PC3: now reaches U1.15 (PC3), U2.18 (PC3)
- net PA0: now reaches U1.16 (~{RESET}/PA0), U2.19 (~{RESET}/PA0)
- net PA1: now reaches U1.17 (PA1), U2.20 (PA1)
- net PA2: now reaches U1.18 (PA2), U2.1 (PA2)
- net PA3: now reaches U1.19 (PA3), U2.2 (PA3)
- net PA4: now reaches U1.2 (PA4), U2.5 (PA4)
- net GND: now reaches U1.20 (GND), U2.21 (GND), U2.3 (GND)
- net PA5: now reaches U1.3 (PA5), U2.6 (PA5)
- net PA6: now reaches U1.4 (PA6), U2.7 (PA6)
- net PA7: now reaches U1.5 (PA7), U2.8 (PA7)
- net PB5: now reaches U1.6 (PB5), U2.9 (PB5)
- net PB5: now also D5.1 (K)
- net PB4: now reaches U1.7 (PB4), U2.10 (PB4)
- net PB4: now also D4.1 (K)
- net PB3: now reaches U1.8 (PB3), U2.11 (PB3)
- net PB3: now also D3.1 (K)
- net PB2: now reaches U1.9 (PB2), U2.12 (PB2)
- net PB2: now also D2.1 (K)
Other:
- moved on the sheet: U1, U2

Commit message: WIP
Parts:
- added C1, C2: 1u, Capacitor_SMD:C_0805_2012Metric, symbol Device:C
- added D8: D_Schottky, symbol Device:D_Schottky
- added J1, J2, J4: Conn_01x02, Connector_Molex:Molex_KK-254_AE-6410-02A_1x02_P2.54mm_Vertical, symbol Connector_Generic:Conn_01x02
- added J3: USB_B_Micro, Connector_USB:USB_Micro-AB_Molex_47590-0001, symbol Connector:USB_B_Micro
- added U3: AMS1117-3.3, Package_TO_SOT_SMD:SOT-223-3_TabPin2, symbol Regulator_Linear:AMS1117-3.3
Connections:
- net +3.3V: now also C1.1, U3.2 (VO)
- net GND: now also C1.2, C2.2, J1.2 (Pin_2), J2.2 (Pin_2), J3.5 (GND), J3.6 (Shield), J4.2 (Pin_2), U3.1 (GND)
- net PB0: now also D4.1 (K); no longer D0.1 (K)
- net PB1: now also D5.1 (K); no longer D1.1 (K)
- net PB2: now also D6.1 (K); no longer D2.1 (K)
- net PB3: now also D7.1 (K); no longer D3.1 (K)
- net PB4: no longer D4.1 (K)
- net PB5: no longer D5.1 (K)
- net PC0: now also D0.1 (K)
- net PC1: now also D1.1 (K)
- net PC2: now also D2.1 (K)
- net PC3: now also D3.1 (K)
- net PA0 renamed ~{RESET}
- net PA1 renamed PA1/MOSI/SDA
- net PA2 renamed PA2/MISO/SCL
- net PA3 renamed PA3/SCK
- net PA4 renamed PA4/SS
- net PA5 renamed PA5/AIN5
- net PA5/AIN5: now also J1.1 (Pin_1)
- net PA6 renamed PA6/OUT
- net PA6/OUT: now also J2.1 (Pin_1)
- new net: D8.2 (A), J3.1 (VBUS)
- new net +VDC: C2.1, D8.1 (K), J4.1 (Pin_1), U3.3 (VI)
- no-connect marks 0 -> 3
Other:
- moved on the sheet: U2
